Commit message: feat: update URDF model to v3 (00-arm-rs_asm-v3)
Co-Authored-By: Claude Fable 5 <noreply@anthropic.com>

File: packages/robot-description/public/robots/rebot-b601-rs/model.urdf (robot description, URDF)
Before this commit: robot 00-arm-rs_asm-v3, 10 links, 9 joints
Links:
- link link2: mass 1.972 -> 1.359
- link link3: mass 1.062 -> 1.0896
- link link4: mass 0.66 -> 0.365
- link link5: mass 0.150120457182895 -> 0.152
- link link6: mass 0.03 -> 0.1
